File: BrushlessMotorDriver_DRV8311.kicad_pcb (KiCad board)
At the start: 2 copper layers, 42 x 35 mm, 33 parts, among them J1 Conn_01x02, J2 Conn_02x04_Odd_Even, J3 Conn_01x16, U1 NJM2864F03, U2 MCP1792T-5002H/CB, U3 PDRV8311HRRWR

Commit message: Add files via upload
Parts:
- added JP7: Jumper, Jumper:SolderJumper-2_P1.3mm_Bridged_RoundedPad1.0x1.5mm, F.Cu at (132.7, 129.5)
- J3: value Conn_01x16 -> Conn_01x18; footprint Connector_PinHeader_2.54mm:PinHeader_1x16_P2.54mm_Vertical -> Connector_PinHeader_2.54mm:PinHeader_1x18_P2.54mm_Vertical
- moved C5 5.39 mm to (156.1, 130.7), turned to -90 degrees
- moved C4 4.21 mm to (153.4, 135.5), turned to 180 degrees
- moved C1 4.04 mm to (153.4, 129.8), turned to 180 degrees
- moved C17 3.28 mm to (157.5, 138.8)
- moved C15 3.20 mm to (162.5, 138.8)
- moved C16 3.20 mm to (160.0, 138.8)
- moved U1 1.16 mm to (153.6, 132.7), turned to 90 degrees
- moved C14 0.40 mm to (135.3, 126.6)
Connections:
- J3 pad 14: SOC -> +3V0
- J3 pad 15: SOB -> SOC
- J3 pad 16: SOA -> SOB
Routing:
- net +3V0: track 13.6 -> 30.4 mm
- net +3V3: track 108.8 -> 104.6 mm
- net SOA: track 36.1 -> 38.6 mm
- net SOB: track 35.3 -> 36.7 mm
- net SOC: track 35.5 -> 34.3 mm
- net GND: track 58.5 -> 59.2 mm
Other:
- board size 42 x 35 mm -> 47 x 35 mm
- board text added: "3V"
- board text added: "BrushlessMotorDriver DRV8311H v.0.2 by Nori"
- board text added: "PhaA"
- board text added: "PhaB"
- board text added: "PhaC"
- board text removed: "BrushlessMotorDriver DRV8311H v.0.1 by Nori"
- board text removed: "PhaseA"
- board text removed: "PhaseB"
- board text removed: "PhaseC"
