File: BrushlessMotorDriver_DRV8311.kicad_sch (KiCad schematic)
At the start: 33 parts, among them J1 Conn_01x02, J2 Conn_02x04_Odd_Even, J3 Conn_01x16, U1 NJM2864F03, U2 MCP1792T-5002H/CB, U3 PDRV8311HRRWR

Commit message: Add files via upload
Parts:
- added JP7: Jumper, Jumper:SolderJumper-2_P1.3mm_Bridged_RoundedPad1.0x1.5mm, symbol Jumper:SolderJumper_2_Bridged
- J3: value Conn_01x16 -> Conn_01x18; footprint Connector_PinHeader_2.54mm:PinHeader_1x16_P2.54mm_Vertical -> Connector_PinHeader_2.54mm:PinHeader_1x18_P2.54mm_Vertical; symbol Connector_Generic:Conn_01x16 -> Connector_Generic:Conn_01x18
Connections:
- net +3V0: now also J3.14 (Pin_14)
- net +3V3: now also JP7.1 (A), JP7.2 (B)
- net GND: now also J3.18 (Pin_18)
- net SOA: now also J3.17 (Pin_17); no longer J3.16 (Pin_16)
- net SOB: now also J3.16 (Pin_16); no longer J3.15 (Pin_15)
- net SOC: now also J3.15 (Pin_15); no longer J3.14 (Pin_14)
Other:
- note added: "Source URL: https://www.tij.co.jp/jp/lit/ds/symlink/drv8311.pdf https://www.shinkoh-faulhaber.jp/JP_data_edition_2020/JP_2214_BXTR_DFF.pdf"
- company: (none) -> Noriaki Nakagawa
- title: (none) -> Brushless Motor Driver DRV8311H
- moved on the sheet: C15, C16, C17
